File: esc_powerboard_kicad_project/power_board.kicad_pcb (KiCad board)
At the start: 2 copper layers, 100.3 x 142.2 mm, 68 parts, among them P1 B+, P2 M-, P3 B-, P4 MOUNT_HOLE, P5 MOUNT_HOLE, P6 MOUNT_HOLE, P7 MOUNT_HOLE, P8 MOUNT_HOLE, Q1 IRFB7437PBF, Q10 IRFB7437PBF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

Commit message: Changed page size to A4 and positioned pcb to page corner
Parts:
- moved C1 157.9 mm to (23.7, 144.9)
- moved C10 157.9 mm to (105.0, 91.6)
- moved C11 157.9 mm to (23.7, 76.3)
- moved C12 157.9 mm to (105.0, 76.3)
- moved C13 157.9 mm to (23.7, 64.9)
- moved C14 157.9 mm to (105.0, 64.9)
- moved C15 157.9 mm to (23.7, 49.7)
- moved C16 157.9 mm to (105.0, 49.7)
- moved C17 157.9 mm to (23.7, 38.2)
- moved C18 157.9 mm to (105.0, 38.2)
- moved C19 157.9 mm to (23.7, 23.0)
- moved C2 157.9 mm to (105.0, 144.9)
- moved C20 157.9 mm to (105.0, 23.0)
- moved C3 157.9 mm to (23.7, 129.7)
- moved C4 157.9 mm to (105.0, 129.7)
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